File: circuits/jelly-kicad/jelly.kicad_sch (KiCad schematic)
At the start: 9 parts, among them J1 Conn_02x07_Counter_Clockwise, U1 28C256, U2 28C256, U3 74LS393, U4 74AHCT273, U5 74AHCT273, U6 74HCT574, U7 74HC245, U8 74LS138

Commit message: Review for make it
Parts:
- removed J1: Conn_02x07_Counter_Clockwise, symbol Connector_Generic:Conn_02x07_Counter_Clockwise
- removed unit 1 of U6
- added J2: Conn_02x08_Counter_Clockwise, symbol Connector_Generic:Conn_02x08_Counter_Clockwise
- added unit 1 of U6
- U4, U5: value 74AHCT273 -> 74AHC574
Connections:
- net CR3: now also U3.6 (Q3)
- net D0: now also U6.2 (Q0)
- net D1: now also U6.5 (Q1)
- net D2: now also U6.6 (Q2)
- net D3: now also U6.9 (Q3)
- net D4: now also U6.12 (Q4)
- net D5: now also U6.15 (Q5)
- net D6: now also U6.16 (Q6)
- net D7: now also U6.19 (Q7)
- net GND: now also J2.1 (Pin_1), J2.8 (Pin_8), U6.10 (GND)
- net T1: now also J2.13 (Pin_13)
- net VCC: now also J2.16 (Pin_16), J2.9 (Pin_9), U6.20 (VCC)
- net /OE6: now also U6.1 (~{Mr})
- net at U7.18 (B0): now also J2.2 (Pin_2)
- net at U7.17 (B1): now also J2.3 (Pin_3)
- net at U7.16 (B2): now also J2.4 (Pin_4)
- net at U7.15 (B3): now also J2.5 (Pin_5)
- net at U7.14 (B4): now also J2.6 (Pin_6)
- net at U7.13 (B5): now also J2.7 (Pin_7)
- net at U7.12 (B6): now also J2.10 (Pin_10)
- net at U7.11 (B7): now also J2.11 (Pin_11)
- net at U2.11 (D0): now also U6.3 (D0)
- net at U2.12 (D1): now also U6.4 (D1)
- net at U2.13 (D2): now also U6.7 (D2)
- net at U2.15 (D3): now also U6.8 (D3)
- net at U2.16 (D4): now also U6.13 (D4)
- net at U2.17 (D5): now also U6.14 (D5)
- net at U2.18 (D6): now also U6.17 (D6)
- net at U2.19 (D7): now also U6.18 (D7)
- net LOOP: now reaches U1.25 (A8)
- net at U4.9 (Q3): now also U1.4 (A6); no longer U1.3 (A7)
- net at U4.6 (Q2): now also U1.5 (A5); no longer U1.4 (A6)
- net at U4.5 (Q1): now also U1.6 (A4); no longer U1.5 (A5)
- net at U4.2 (Q0): now also U1.7 (A3); no longer U1.6 (A4)
- net M0 renamed C4
- net M1 renamed C5
- net M2 renamed C6
- net M3 renamed C7
- net C7: now also U6.11 (Cp)
- net T0 renamed C0
- net C0: now also J2.12 (Pin_12)
- net T2 renamed C2
- net C2: now also J2.14 (Pin_14)
- net T3 renamed C3
- net C3: now also J2.15 (Pin_15)
- new net ZERO: U1.3 (A7)
- no-connect marks 17 -> 16
Other:
- moved on the sheet: U1, U2, U3A, U3B, U4, U5, U6C, U7, U8
